File: aux-pcb/airdisk.kicad_pcb (KiCad board)
At the start: 2 copper layers, 78.7 x 31.1 mm, 52 parts, among them U1 USBLC6-2SC6

Commit message: update pcb
Parts:
- removed D1: LED, Diode_SMD:D_0603_1608Metric_Pad1.05x0.95mm_HandSolder
- removed TP2: TestPoint, airdisk:TE_3-2199250-5
- added R5: 0R, Resistor_SMD:R_0402_1005Metric, B.Cu at (139.1, 61.0)
- added REF**: TE_3-2199250-5, airdisk:TE_3-2199250-5, B.Cu at (114.3, 73.0)
- TP1: footprint airdisk:TE_3-2199250-5 -> TestPoint:TestPoint_Pad_D1.5mm; moved to F.Cu
- moved TP1 13.9 mm to (139.7, 66.7)
- moved TP12 1.27 mm to (152.4, 54.6)
Connections:
- C7 pad 1: Net-(2V1-Pad1) -> Net-(C7-Pad1)
- ETH1 pad P5: Net-(2V1-Pad1) -> Net-(C7-Pad1)
- ETH1 pad P6: Net-(2V1-Pad1) -> Net-(C7-Pad1)
- TE11 pad 1: Net-(2V1-Pad1) -> Net-(C7-Pad1)
- TP1 pad 1: Net-(D1-Pad2) -> Net-(2V1-Pad1)
Routing:
- net Net-(C7-Pad1): track 0.00 -> 37.6 mm, vias 0 -> 1
- net Net-(2V1-Pad1): track 40.0 -> 6.41 mm
- net /VBUS: track 37.7 -> 29.8 mm
- net Net-(D1-Pad2): track 3.91 -> 0.00 mm, vias 1 -> 0
- net Earth: track 75.5 -> 78.0 mm, vias 109 -> 106
- net Net-(TP11-Pad1): track 4.97 -> 4.44 mm
